File: s3t.sch (KiCad schematic (older format))
At the start: 65 parts

Commit message: change TF card
Parts:
- removed R? (x6): R, symbol R
- added J?: Conn_01x02, symbol Conn_01x02
- added R? (x2): R, symbol R
- C?: value CP -> 47uF
Connections:
- net labels added: LCD_EN, LCD_PWM, SD_CD
- net labels removed: LCD_BL
- wire segments 402 -> 474

Commit message: add some lib
Parts:
- C1, C5: renamed from C?; footprint (none) -> Capacitors_SMD:C_0805
- C10, C14, C17, C18, C19, C2, C4, C9: renamed from C?; footprint (none) -> Capacitors_SMD:C_0603
- C3: renamed from C?; footprint (none) -> Resistors_SMD:R_0603
- C6: renamed from C?; footprint (none) -> Capacitors_THT:CP_Radial_D8.0mm_P2.50mm
- C7, C8: renamed from C?; value C -> 7pF; footprint (none) -> Capacitors_SMD:C_0603
- D1, D2: renamed from D?; footprint (none) -> TO_SOT_Packages_SMD:SOT-23
- D3, D4, D5: renamed from D?; footprint (none) -> LEDs:LED_0805
- D6: renamed from D?; footprint (none) -> Diodes_SMD:D_1206
- J3: renamed from J?; footprint (none) -> Connectors:USB_Mini-B
- L1: renamed from L?; footprint (none) -> Inductors_SMD:L_7.3x7.3_H3.5
- L2: renamed from L?; footprint (none) -> Inductors_SMD:L_1812
- R1, R10, R12, R14, R17, R2, R3, R4, R5, R6, R7, R8, R9: renamed from R?; footprint (none) -> Resistors_SMD:R_0603
- R18: renamed from R?; footprint (none) -> Capacitors_SMD:C_0603
- U1: renamed from U?; footprint (none) -> TO_SOT_Packages_SMD:SOT-223
- U2: renamed from U?; footprint (none) -> tfcard:tfcard
- U3: renamed from U?; footprint (none) -> s3core:S3Core
- U4, U5: renamed from U?; footprint (none) -> TO_SOT_Packages_SMD:SOT-23-6
- U6: renamed from U?; footprint (none) -> fpc36:Hirose_FH12-36S-0.5SH_1x36-1MP_P0.50mm_Horizontal
- U7: renamed from U?; footprint (none) -> fpc40:Hirose_FH12-40S-0.5SH_1x40-1MP_P0.50mm_Horizontal
- gave numbers to parts that had none: 18
Connections:
- net labels added: TEN
- wire segments 474 -> 403

Commit message: update pcb lib
Parts:
- C15: footprint (none) -> Capacitors_SMD:C_0603
- C3: value C -> 0.1uF; footprint Resistors_SMD:R_0603 -> Capacitors_SMD:C_0603
- J1: footprint (none) -> Connectors_JST:JST_EH_B04B-EH-A_04x2.50mm_Straight
- L1: footprint Inductors_SMD:L_7.3x7.3_H3.5 -> Inductors_SMD:L_1812
- R15, R16: footprint (none) -> Resistors_SMD:R_0805
- R6: value R -> 10K
- SW1, SW2, SW3, SW4, SW5, SW6: footprint (none) -> tfcard:button
Connections:
- wire segments 403 -> 399

Commit message: update pcb route
Parts:
- added AE?: Antenna, symbol Antenna
- added J4, J5, J6, J7: HOLE, hole:hole, symbol TEST_1P
- C11, C12, C16: footprint (none) -> Capacitors_SMD:C_0603
- D6: footprint Diodes_SMD:D_1206 -> Diodes_SMD:D_SMA
- D7: footprint (none) -> Diodes_SMD:D_SMA
- J2: footprint (none) -> Connectors_JST:JST_EH_B02B-EH-A_02x2.50mm_Straight
- R11, R13: footprint (none) -> Resistors_SMD:R_0603
Connections:
- wire segments 399 -> 406
- no-connect marks 0 -> 51
Changed lines of the file:
@@
 	1    0    0    -1
 $EndComp
-Text Label 12300 8100 0    60   ~ 0
+Text Label 12450 8100 0    60   ~ 0
 USBDP
-Text Label 12300 8200 0    60   ~ 0
+Text Label 12450 8200 0    60   ~ 0
 USBDN
 Text Label 14900 7850 0    60   ~ 0
@@
 F 0 "D6" H 21200 17050 50  0000 C CNN
 F 1 "D" H 21200 16850 50  0000 C CNN
-F 2 "Diodes_SMD:D_1206" H 21200 16950 50  0001 C CNN
+F 2 "Diodes_SMD:D_SMA" H 21200 16950 50  0001 C CNN
 F 3 "" H 21200 16950 50  0001 C CNN
 	1    21200 16950
@@
 F 0 "D7" H 21350 12600 50  0000 C CNN
 F 1 "D" H 21350 12400 50  0000 C CNN
-F 2 "" H 21350 12500 50  0001 C CNN
+F 2 "Diodes_SMD:D_SMA" H 21350 12500 50  0001 C CNN
 F 3 "" H 21350 12500 50  0001 C CNN
 	1    21350 12500
@@
 F 0 "C11" H 21125 13500 50  0000 L CNN
 F 1 "0.1uF" H 21125 13300 50  0000 L CNN
-F 2 "" H 21138 13250 50  0001 C CNN
+F 2 "Capacitors_SMD:C_0603" H 21138 13250 50  0001 C CNN
 F 3 "" H 21100 13400 50  0001 C CNN
 	1    21100 13400
@@
 F 0 "C12" H 21625 13500 50  0000 L CNN
 F 1 "0.1uF" H 21625 13300 50  0000 L CNN
-F 2 "" H 21638 13250 50  0001 C CNN
+F 2 "Capacitors_SMD:C_0603" H 21638 13250 50  0001 C CNN
 F 3 "" H 21600 13400 50  0001 C CNN
 	1    21600 13400
@@
 F 0 "R11" V 19980 14750 50  0000 C CNN
 F 1 "5R1" V 19900 14750 50  0000 C CNN
-F 2 "" V 19830 14750 50  0001 C CNN
+F 2 "Resistors_SMD:R_0603" V 19830 14750 50  0001 C CNN
 F 3 "" H 19900 14750 50  0001 C CNN
 	1    19900 14750
@@
 F 0 "C16" H 22325 12850 50  0000 L CNN
 F 1 "0.1uF" H 22325 12650 50  0000 L CNN
-F 2 "" H 22338 12600 50  0001 C CNN
+F 2 "Capacitors_SMD:C_0603" H 22338 12600 50  0001 C CNN
 F 3 "" H 22300 12750 50  0001 C CNN
 	1    22300 12750
@@
 	11150 7900 11250 7900
 Wire Wire Line
-	11250 6950 11250 7900
+	11250 7900 11250 6950
 Wire Wire Line
 	11750 6950 11750 6500
@@
 	15200 9550 14800 9550
 Wire Wire Line
-	15200 9650 14800 9650
+	13900 9650 15200 9650
 Wire Wire Line
 	15200 9750 14800 9750
@@
 	23000 5500 22450 5500
 Wire Wire Line
-	22450 5700 22450 5500
+	22450 5500 22450 5700
 Wire Wire Line
 	22450 5600 23000 5600
@@
 $EndComp
 $Comp
-L GND #PWR024
+L GND #PWR023
 U 1 1 5D5250A0
 P 12050 13900
-F 0 "#PWR024" H 12050 13650 50  0001 C CNN
+F 0 "#PWR023" H 12050 13650 50  0001 C CNN
 F 1 "GND" H 12050 13750 50  0000 C CNN
 F 2 "" H 12050 13900 50  0001 C CNN
@@
 	14400 13450 14350 13450
 $Comp
-L +3.3V #PWR025
+L +3.3V #PWR024
 U 1 1 5D525D0A
 P 13550 12200
-F 0 "#PWR025" H 13550 12050 50  0001 C CNN
+F 0 "#PWR024" H 13550 12050 50  0001 C CNN
 F 1 "+3.3V" H 13550 12340 50  0000 C CNN
 F 2 "" H 13550 12200 50  0001 C CNN
@@
 	26200 12950 26450 12950
 $Comp
-L GND #PWR026
+L GND #PWR025
 U 1 1 5D51A5B9
 P 25600 12900
-F 0 "#PWR026" H 25600 12650 50  0001 C CNN
+F 0 "#PWR025" H 25600 12650 50  0001 C CNN
 F 1 "GND" H 25600 12750 50  0000 C CNN
 F 2 "" H 25600 12900 50  0001 C CNN
@@
 	26250 13750 26450 13750
 $Comp
-L GND #PWR027
+L GND #PWR026
 U 1 1 5D51B696
 P 25600 13700
-F 0 "#PWR027" H 25600 13450 50  0001 C CNN
+F 0 "#PWR026" H 25600 13450 50  0001 C CNN
 F 1 "GND" H 25600 13550 50  0000 C CNN
 F 2 "" H 25600 13700 50  0001 C CNN
@@
 	26450 15150 25800 15150
 $Comp
-L GND #PWR028
+L GND #PWR027
 U 1 1 5D51D89D
 P 25600 14500
-F 0 "#PWR028" H 25600 14250 50  0001 C CNN
+F 0 "#PWR027" H 25600 14250 50  0001 C CNN
 F 1 "GND" H 25600 14350 50  0000 C CNN
 F 2 "" H 25600 14500 50  0001 C CNN
@@
 Connection ~ 26250 14500
 $Comp
-L GND #PWR029
+L GND #PWR028
 U 1 1 5D51DE1A
 P 25600 15250
-F 0 "#PWR029" H 25600 15000 50  0001 C CNN
+F 0 "#PWR028" H 25600 15000 50  0001 C CNN
 F 1 "GND" H 25600 15100 50  0000 C CNN
 F 2 "" H 25600 15250 50  0001 C CNN
@@
 LCD_DE
 $Comp
-L GND #PWR030
+L GND #PWR029
 U 1 1 5D520BC1
 P 25400 15950
-F 0 "#PWR030" H 25400 15700 50  0001 C CNN
+F 0 "#PWR029" H 25400 15700 50  0001 C CNN
 F 1 "GND" H 25400 15800 50  0000 C CNN
 F 2 "" H 25400 15950 50  0001 C CNN
@@
 	25600 15700 25500 15700
 $Comp
-L +3.3V #PWR031
+L +3.3V #PWR030
 U 1 1 5D521E0E
 P 24700 15400
-F 0 "#PWR031" H 24700 15250 50  0001 C CNN
+F 0 "#PWR030" H 24700 15250 50  0001 C CNN
 F 1 "+3.3V" H 24700 15540 50  0000 C CNN
 F 2 "" H 24700 15400 50  0001 C CNN
@@
 $EndComp
 $Comp
-L +3.3V #PWR032
+L +3.3V #PWR031
 U 1 1 5D5254AD
 P 27900 13600
-F 0 "#PWR032" H 27900 13450 50  0001 C CNN
+F 0 "#PWR031" H 27900 13450 50  0001 C CNN
 F 1 "+3.3V" H 27900 13740 50  0000 C CNN
 F 2 "" H 27900 13600 50  0001 C CNN
@@
 $EndComp
 $Comp
-L +3.3V #PWR033
+L +3.3V #PWR032
 U 1 1 5D525543
 P 28350 13600
-F 0 "#PWR033" H 28350 13450 50  0001 C CNN
+F 0 "#PWR032" H 28350 13450 50  0001 C CNN
 F 1 "+3.3V" H 28350 13740 50  0000 C CNN
 F 2 "" H 28350 13600 50  0001 C CNN
@@
 $EndComp
 $Comp
-L GND #PWR034
+L GND #PWR033
 U 1 1 5D52565B
 P 27900 14600
-F 0 "#PWR034" H 27900 14350 50  0001 C CNN
+F 0 "#PWR033" H 27900 14350 50  0001 C CNN
 F 1 "GND" H 27900 14450 50  0000 C CNN
 F 2 "" H 27900 14600 50  0001 C CNN
@@
 $EndComp
 $Comp
-L GND #PWR035
+L GND #PWR034
 U 1 1 5D5256F1
 P 28350 14600
-F 0 "#PWR035" H 28350 14350 50  0001 C CNN
+F 0 "#PWR034" H 28350 14350 50  0001 C CNN
 F 1 "GND" H 28350 14450 50  0000 C CNN
 F 2 "" H 28350 14600 50  0001 C CNN
@@
 F 0 "J2" H 10000 7050 50  0000 C CNN
 F 1 "Conn_01x02" H 10000 6750 50  0000 C CNN
-F 2 "" H 10000 6950 50  0001 C CNN
+F 2 "Connectors_JST:JST_EH_B02B-EH-A_02x2.50mm_Straight" H 10000 6950 50  0001 C CNN
 F 3 "" H 10000 6950 50  0001 C CNN
 	1    10000 6950
@@
 $EndComp
 $Comp
-L GND #PWR036
+L GND #PWR035
 U 1 1 5D52FA71
 P 10250 7450
-F 0 "#PWR036" H 10250 7200 50  0001 C CNN
+F 0 "#PWR035" H 10250 7200 50  0001 C CNN
 F 1 "GND" H 10250 7300 50  0000 C CNN
 F 2 "" H 10250 7450 50  0001 C CNN
@@
 F 0 "R13" V 21630 14500 50  0000 C CNN
 F 1 "R" V 21550 14500 50  0000 C CNN
-F 2 "" V 21480 14500 50  0001 C CNN
+F 2 "Resistors_SMD:R_0603" V 21480 14500 50  0001 C CNN
 F 3 "" H 21550 14500 50  0001 C CNN
 	1    21550 14500
@@
 Connection ~ 21550 14250
 $Comp
-L GND #PWR037
+L GND #PWR036
 U 1 1 5D53AA83
 P 21550 14900
-F 0 "#PWR037" H 21550 14650 50  0001 C CNN
+F 0 "#PWR036" H 21550 14650 50  0001 C CNN
 F 1 "GND" H 21550 14750 50  0000 C CNN
 F 2 "" H 21550 14900 50  0001 C CNN
@@
 	8000 11550 7750 11550
 Connection ~ 7750 11650
+NoConn ~ 14800 8250
+NoConn ~ 14800 7750
+NoConn ~ 14800 8450
+NoConn ~ 14800 8550
+NoConn ~ 14800 8650
+NoConn ~ 14800 8750
+NoConn ~ 14800 8850
+NoConn ~ 14800 8950
+NoConn ~ 14800 9050
+NoConn ~ 14800 9150
+NoConn ~ 14800 9250
+NoConn ~ 14800 9350
+NoConn ~ 14800 9450
+NoConn ~ 14800 9850
+NoConn ~ 14800 9950
+NoConn ~ 17950 11350
+NoConn ~ 18450 11350
+NoConn ~ 18550 11350
+NoConn ~ 19950 8050
+NoConn ~ 19950 7950
+NoConn ~ 19950 7850
+NoConn ~ 19950 7750
+NoConn ~ 19950 7650
+NoConn ~ 19950 7550
+NoConn ~ 19950 7450
+NoConn ~ 16700 6450
+NoConn ~ 16800 6450
+NoConn ~ 16900 6450
+NoConn ~ 17000 6450
+NoConn ~ 17100 6450
+NoConn ~ 17200 6450
+NoConn ~ 17300 6450
+NoConn ~ 17400 6450
+NoConn ~ 17500 6450
+NoConn ~ 17600 6450
+NoConn ~ 17700 6450
+NoConn ~ 17800 6450
+NoConn ~ 17900 6450
+NoConn ~ 18000 6450
+NoConn ~ 18100 6450
+NoConn ~ 18200 6450
+NoConn ~ 18300 6450
+NoConn ~ 18400 6450
+NoConn ~ 18500 6450
+NoConn ~ 18600 6450
+NoConn ~ 18700 6450
+NoConn ~ 18800 6450
+NoConn ~ 23000 5700
+NoConn ~ 23000 5800
+NoConn ~ 23000 6100
+NoConn ~ 23000 6200
+$Comp
+L TEST_1P J4
+U 1 1 5D597B7A
+P 11150 19750
+F 0 "J4" H 11150 20020 50  0000 C CNN
+F 1 "HOLE" H 11150 19950 50  0000 C CNN
+F 2 "hole:hole" H 11350 19750 50  0001 C CNN
+F 3 "" H 11350 19750 50  0001 C CNN
+	1    11150 19750
+	1    0    0    -1
+$EndComp
+$Comp
+L TEST_1P J5
+U 1 1 5D597DA8
+P 11550 19750
+F 0 "J5" H 11550 20020 50  0000 C CNN
+F 1 "HOLE" H 11550 19950 50  0000 C CNN
+F 2 "hole:hole" H 11750 19750 50  0001 C CNN
+F 3 "" H 11750 19750 50  0001 C CNN
+	1    11550 19750
+	1    0    0    -1
+$EndComp
+$Comp
+L TEST_1P J6
+U 1 1 5D597E53
+P 11950 19750
+F 0 "J6" H 11950 20020 50  0000 C CNN
+F 1 "HOLE" H 11950 19950 50  0000 C CNN
+F 2 "hole:hole" H 12150 19750 50  0001 C CNN
+F 3 "" H 12150 19750 50  0001 C CNN
+	1    11950 19750
+	1    0    0    -1
+$EndComp
+$Comp
+L TEST_1P J7
+U 1 1 5D597EF8
+P 12350 19750
+F 0 "J7" H 12350 20020 50  0000 C CNN
+F 1 "HOLE" H 12350 19950 50  0000 C CNN
+F 2 "hole:hole" H 12550 19750 50  0001 C CNN
+F 3 "" H 12550 19750 50  0001 C CNN
+	1    12350 19750
+	1    0    0    -1
+$EndComp
+$Comp
+L GND #PWR037
+U 1 1 5D5982D2
+P 11750 20050
+F 0 "#PWR037" H 11750 19800 50  0001 C CNN
+F 1 "GND" H 11750 19900 50  0000 C CNN
+F 2 "" H 11750 20050 50  0001 C CNN
+F 3 "" H 11750 20050 50  0001 C CNN
+	1    11750 20050
+	1    0    0    -1
+$EndComp
+Wire Wire Line
+	11150 19750 11150 19900
+Wire Wire Line
+	11150 19900 12350 19900
+Wire Wire Line
+	12350 19900 12350 19750
+Wire Wire Line
+	11950 19750 11950 19900
+Connection ~ 11950 19900
+Wire Wire Line
+	11550 19750 11550 19900
+Connection ~ 11550 19900
+Wire Wire Line
+	11750 19900 11750 20050
+Connection ~ 11750 19900
+$Comp
+L Antenna AE?
+U 1 1 5D5A75DA
+P 13900 9350
+F 0 "AE?" H 13825 9425 50  0000 R CNN
+F 1 "Antenna" H 13825 9350 50  0000 R CNN
+F 2 "" H 13900 9350 50  0001 C CNN
+F 3 "" H 13900 9350 50  0001 C CNN
+	1    13900 9350
+	1    0    0    -1
+$EndComp
+Wire Wire Line
+	13900 9650 13900 9550
 $EndSCHEMATC
