File: _saved_s3t.sch (KiCad schematic (older format))
At the start: 67 parts, among them J1 DEBUG_UART0, J2 Conn_01x02, J3 USB_OTG, J4 HOLE, J5 HOLE, J6 HOLE, J7 HOLE, SW1 SW_DIP_x01, SW2 SW_DIP_x01, SW3 SW_DIP_x01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

Commit message: update pcb
Parts:
- gave numbers to parts that had none: 1
Changed lines of the file:
@@
 $EndComp
 $Comp
-L GND #PWR01
+L GND #PWR12
 U 1 1 5D471CFA
 P 11200 9050
-F 0 "#PWR01" H 11200 8800 50  0001 C CNN
+F 0 "#PWR12" H 11200 8800 50  0001 C CNN
 F 1 "GND" H 11200 8900 50  0000 C CNN
 F 2 "" H 11200 9050 50  0001 C CNN
@@
 $EndComp
 $Comp
-L +5V #PWR02
+L +5V #PWR13
 U 1 1 5D471D38
 P 11750 6500
-F 0 "#PWR02" H 11750 6350 50  0001 C CNN
+F 0 "#PWR13" H 11750 6350 50  0001 C CNN
 F 1 "+5V" H 11750 6640 50  0000 C CNN
 F 2 "" H 11750 6500 50  0001 C CNN
@@
 5V
 $Comp
-L GND #PWR03
+L GND #PWR11
 U 1 1 5D471DD3
 P 10650 7400
-F 0 "#PWR03" H 10650 7150 50  0001 C CNN
+F 0 "#PWR11" H 10650 7150 50  0001 C CNN
 F 1 "GND" H 10650 7250 50  0000 C CNN
 F 2 "" H 10650 7400 50  0001 C CNN
@@
 $EndComp
 $Comp
-L GND #PWR04
+L GND #PWR5
 U 1 1 5D4986ED
 P 6400 17500
-F 0 "#PWR04" H 6400 17250 50  0001 C CNN
+F 0 "#PWR5" H 6400 17250 50  0001 C CNN
 F 1 "GND" H 6400 17350 50  0000 C CNN
 F 2 "" H 6400 17500 50  0001 C CNN
@@
 $EndComp
 $Comp
-L +3.3V #PWR05
+L +3.3V #PWR1
 U 1 1 5D4993F0
 P 4700 14600
-F 0 "#PWR05" H 4700 14450 50  0001 C CNN
+F 0 "#PWR1" H 4700 14450 50  0001 C CNN
 F 1 "+3.3V" H 4700 14740 50  0000 C CNN
 F 2 "" H 4700 14600 50  0001 C CNN
@@
 $EndComp
 $Comp
-L GND #PWR06
+L GND #PWR4
 U 1 1 5D49AB62
 P 6300 15400
-F 0 "#PWR06" H 6300 15150 50  0001 C CNN
+F 0 "#PWR4" H 6300 15150 50  0001 C CNN
 F 1 "GND" H 6300 15250 50  0000 C CNN
 F 2 "" H 6300 15400 50  0001 C CNN
@@
 $EndComp
 $Comp
-L +5V #PWR07
+L +5V #PWR2
 U 1 1 5D49B558
 P 5350 9900
-F 0 "#PWR07" H 5350 9750 50  0001 C CNN
+F 0 "#PWR2" H 5350 9750 50  0001 C CNN
 F 1 "+5V" H 5350 10040 50  0000 C CNN
 F 2 "" H 5350 9900 50  0001 C CNN
@@
 $EndComp
 $Comp
-L GND #PWR08
+L GND #PWR3
 U 1 1 5D49B87A
 P 5350 10650
-F 0 "#PWR08" H 5350 10400 50  0001 C CNN
+F 0 "#PWR3" H 5350 10400 50  0001 C CNN
 F 1 "GND" H 5350 10500 50  0000 C CNN
 F 2 "" H 5350 10650 50  0001 C CNN
@@
 $EndComp
 $Comp
-L GND #PWR09
+L GND #PWR8
 U 1 1 5D4ED4A6
 P 8400 8950
-F 0 "#PWR09" H 8400 8700 50  0001 C CNN
+F 0 "#PWR8" H 8400 8700 50  0001 C CNN
 F 1 "GND" H 8400 8800 50  0000 C CNN
 F 2 "" H 8400 8950 50  0001 C CNN
@@
 $EndComp
 $Comp
-L +5V #PWR010
+L +5V #PWR6
 U 1 1 5D4EDBD2
 P 6450 7100
-F 0 "#PWR010" H 6450 6950 50  0001 C CNN
+F 0 "#PWR6" H 6450 6950 50  0001 C CNN
 F 1 "+5V" H 6450 7240 50  0000 C CNN
 F 2 "" H 6450 7100 50  0001 C CNN
@@
 $EndComp
 $Comp
-L GND #PWR011
+L GND #PWR19
 U 1 1 5D4F2708
 P 18950 18350
-F 0 "#PWR011" H 18950 18100 50  0001 C CNN
+F 0 "#PWR19" H 18950 18100 50  0001 C CNN
 F 1 "GND" H 18950 18200 50  0000 C CNN
 F 2 "" H 18950 18350 50  0001 C CNN
@@
 $EndComp
 $Comp
-L GND #PWR012
+L GND #PWR26
 U 1 1 5D4F3151
 P 22100 18300
-F 0 "#PWR012" H 22100 18050 50  0001 C CNN
+F 0 "#PWR26" H 22100 18050 50  0001 C CNN
 F 1 "GND" H 22100 18150 50  0000 C CNN
 F 2 "" H 22100 18300 50  0001 C CNN
@@
 $EndComp
 $Comp
-L GND #PWR013
+L GND #PWR20
 U 1 1 5D4F4949
 P 19900 15200
-F 0 "#PWR013" H 19900 14950 50  0001 C CNN
+F 0 "#PWR20" H 19900 14950 50  0001 C CNN
 F 1 "GND" H 19900 15050 50  0000 C CNN
 F 2 "" H 19900 15200 50  0001 C CNN
@@
 $EndComp
 $Comp
-L GND #PWR014
+L GND #PWR21
 U 1 1 5D4F4F24
 P 21350 13700
-F 0 "#PWR014" H 21350 13450 50  0001 C CNN
+F 0 "#PWR21" H 21350 13450 50  0001 C CNN
 F 1 "GND" H 21350 13550 50  0000 C CNN
 F 2 "" H 21350 13700 50  0001 C CNN
@@
 LCD_EN
 $Comp
-L GND #PWR015
+L GND #PWR27
 U 1 1 5D4F6FFD
 P 22300 13250
-F 0 "#PWR015" H 22300 13000 50  0001 C CNN
+F 0 "#PWR27" H 22300 13000 50  0001 C CNN
 F 1 "GND" H 22300 13100 50  0000 C CNN
 F 2 "" H 22300 13250 50  0001 C CNN
@@
 $EndComp
 $Comp
-L +5V #PWR016
+L +5V #PWR22
 U 1 1 5D4F7D49
 P 21400 12950
-F 0 "#PWR016" H 21400 12800 50  0001 C CNN
+F 0 "#PWR22" H 21400 12800 50  0001 C CNN
 F 1 "+5V" H 21400 13090 50  0000 C CNN
 F 2 "" H 21400 12950 50  0001 C CNN
@@
 $EndComp
 $Comp
-L GND #PWR017
+L GND #PWR17
 U 1 1 5D4FA77D
 P 12150 9150
-F 0 "#PWR017" H 12150 8900 50  0001 C CNN
+F 0 "#PWR17" H 12150 8900 50  0001 C CNN
 F 1 "GND" H 12150 9000 50  0000 C CNN
 F 2 "" H 12150 9150 50  0001 C CNN
@@
 $EndComp
 $Comp
-L GND #PWR018
+L GND #PWR16
 U 1 1 5D4FA991
 P 12100 7700
-F 0 "#PWR018" H 12100 7450 50  0001 C CNN
+F 0 "#PWR16" H 12100 7450 50  0001 C CNN
 F 1 "GND" H 12100 7550 50  0000 C CNN
 F 2 "" H 12100 7700 50  0001 C CNN
@@
 SD_DAT3
 $Comp
-L +3.3V #PWR019
+L +3.3V #PWR9
 U 1 1 5D503744
 P 10000 12550
-F 0 "#PWR019" H 10000 12400 50  0001 C CNN
+F 0 "#PWR9" H 10000 12400 50  0001 C CNN
 F 1 "+3.3V" H 10000 12690 50  0000 C CNN
 F 2 "" H 10000 12550 50  0001 C CNN
@@
 $EndComp
 $Comp
-L GND #PWR020
+L GND #PWR7
 U 1 1 5D503A5B
 P 8050 12500
-F 0 "#PWR020" H 8050 12250 50  0001 C CNN
+F 0 "#PWR7" H 8050 12250 50  0001 C CNN
 F 1 "GND" H 8050 12350 50  0000 C CNN
 F 2 "" H 8050 12500 50  0001 C CNN
@@
 Connection ~ 22250 5700
 $Comp
-L GND #PWR021
+L GND #PWR25
 U 1 1 5D510B47
 P 22100 5750
-F 0 "#PWR021" H 22100 5500 50  0001 C CNN
+F 0 "#PWR25" H 22100 5500 50  0001 C CNN
 F 1 "GND" H 22100 5600 50  0000 C CNN
 F 2 "" H 22100 5750 50  0001 C CNN
@@
 Connection ~ 22300 8400
 $Comp
-L GND #PWR022
+L GND #PWR24
 U 1 1 5D51A273
 P 22000 8250
-F 0 "#PWR022" H 22000 8000 50  0001 C CNN
+F 0 "#PWR24" H 22000 8000 50  0001 C CNN
 F 1 "GND" H 22000 8100 50  0000 C CNN
 F 2 "" H 22000 8250 50  0001 C CNN
@@
 $EndComp
 $Comp
-L GND #PWR023
+L GND #PWR15
 U 1 1 5D5250A0
 P 12050 13900
-F 0 "#PWR023" H 12050 13650 50  0001 C CNN
+F 0 "#PWR15" H 12050 13650 50  0001 C CNN
 F 1 "GND" H 12050 13750 50  0000 C CNN
 F 2 "" H 12050 13900 50  0001 C CNN
@@
 	14400 13450 14350 13450
 $Comp
-L +3.3V #PWR024
+L +3.3V #PWR18
 U 1 1 5D525D0A
 P 13550 12200
-F 0 "#PWR024" H 13550 12050 50  0001 C CNN
+F 0 "#PWR18" H 13550 12050 50  0001 C CNN
 F 1 "+3.3V" H 13550 12340 50  0000 C CNN
 F 2 "" H 13550 12200 50  0001 C CNN
@@
 	26200 12950 26450 12950
 $Comp
-L GND #PWR025
+L GND #PWR30
 U 1 1 5D51A5B9
 P 25600 12900
-F 0 "#PWR025" H 25600 12650 50  0001 C CNN
+F 0 "#PWR30" H 25600 12650 50  0001 C CNN
 F 1 "GND" H 25600 12750 50  0000 C CNN
 F 2 "" H 25600 12900 50  0001 C CNN
@@
 	26250 13750 26450 13750
 $Comp
-L GND #PWR026
+L GND #PWR31
 U 1 1 5D51B696
 P 25600 13700
-F 0 "#PWR026" H 25600 13450 50  0001 C CNN
+F 0 "#PWR31" H 25600 13450 50  0001 C CNN
 F 1 "GND" H 25600 13550 50  0000 C CNN
 F 2 "" H 25600 13700 50  0001 C CNN
@@
 	26450 15150 25800 15150
 $Comp
-L GND #PWR027
+L GND #PWR32
 U 1 1 5D51D89D
 P 25600 14500
-F 0 "#PWR027" H 25600 14250 50  0001 C CNN
+F 0 "#PWR32" H 25600 14250 50  0001 C CNN
 F 1 "GND" H 25600 14350 50  0000 C CNN
 F 2 "" H 25600 14500 50  0001 C CNN
@@
 Connection ~ 26250 14500
 $Comp
-L GND #PWR028
+L GND #PWR33
 U 1 1 5D51DE1A
 P 25600 15250
-F 0 "#PWR028" H 25600 15000 50  0001 C CNN
+F 0 "#PWR33" H 25600 15000 50  0001 C CNN
 F 1 "GND" H 25600 15100 50  0000 C CNN
 F 2 "" H 25600 15250 50  0001 C CNN
@@
 LCD_DE
 $Comp
-L GND #PWR029
+L GND #PWR29
 U 1 1 5D520BC1
 P 25400 15950
-F 0 "#PWR029" H 25400 15700 50  0001 C CNN
+F 0 "#PWR29" H 25400 15700 50  0001 C CNN
 F 1 "GND" H 25400 15800 50  0000 C CNN
 F 2 "" H 25400 15950 50  0001 C CNN
@@
 	25600 15700 25500 15700
 $Comp
-L +3.3V #PWR030
+L +3.3V #PWR28
 U 1 1 5D521E0E
 P 24700 15400
-F 0 "#PWR030" H 24700 15250 50  0001 C CNN
+F 0 "#PWR28" H 24700 15250 50  0001 C CNN
 F 1 "+3.3V" H 24700 15540 50  0000 C CNN
 F 2 "" H 24700 15400 50  0001 C CNN
@@
 $EndComp
 $Comp
-L +3.3V #PWR031
+L +3.3V #PWR34
 U 1 1 5D5254AD
 P 27900 13600
-F 0 "#PWR031" H 27900 13450 50  0001 C CNN
+F 0 "#PWR34" H 27900 13450 50  0001 C CNN
 F 1 "+3.3V" H 27900 13740 50  0000 C CNN
 F 2 "" H 27900 13600 50  0001 C CNN
@@
 $EndComp
 $Comp
-L +3.3V #PWR032
+L +3.3V #PWR36
 U 1 1 5D525543
 P 28350 13600
-F 0 "#PWR032" H 28350 13450 50  0001 C CNN
+F 0 "#PWR36" H 28350 13450 50  0001 C CNN
 F 1 "+3.3V" H 28350 13740 50  0000 C CNN
 F 2 "" H 28350 13600 50  0001 C CNN
@@
 $EndComp
 $Comp
-L GND #PWR033
+L GND #PWR35
 U 1 1 5D52565B
 P 27900 14600
-F 0 "#PWR033" H 27900 14350 50  0001 C CNN
+F 0 "#PWR35" H 27900 14350 50  0001 C CNN
 F 1 "GND" H 27900 14450 50  0000 C CNN
 F 2 "" H 27900 14600 50  0001 C CNN
@@
 $EndComp
 $Comp
-L GND #PWR034
+L GND #PWR37
 U 1 1 5D5256F1
 P 28350 14600
-F 0 "#PWR034" H 28350 14350 50  0001 C CNN
+F 0 "#PWR37" H 28350 14350 50  0001 C CNN
 F 1 "GND" H 28350 14450 50  0000 C CNN
 F 2 "" H 28350 14600 50  0001 C CNN
@@
 $EndComp
 $Comp
-L GND #PWR035
+L GND #PWR10
 U 1 1 5D52FA71
 P 10250 7450
-F 0 "#PWR035" H 10250 7200 50  0001 C CNN
+F 0 "#PWR10" H 10250 7200 50  0001 C CNN
 F 1 "GND" H 10250 7300 50  0000 C CNN
 F 2 "" H 10250 7450 50  0001 C CNN
@@
 Connection ~ 21550 14250
 $Comp
-L GND #PWR036
+L GND #PWR23
 U 1 1 5D53AA83
 P 21550 14900
-F 0 "#PWR036" H 21550 14650 50  0001 C CNN
+F 0 "#PWR23" H 21550 14650 50  0001 C CNN
 F 1 "GND" H 21550 14750 50  0000 C CNN
 F 2 "" H 21550 14900 50  0001 C CNN
@@
 $EndComp
 $Comp
-L GND #PWR037
+L GND #PWR14
 U 1 1 5D5982D2
 P 11750 20050
-F 0 "#PWR037" H 11750 19800 50  0001 C CNN
+F 0 "#PWR14" H 11750 19800 50  0001 C CNN
 F 1 "GND" H 11750 19900 50  0000 C CNN
 F 2 "" H 11750 20050 50  0001 C CNN
@@
 Connection ~ 11750 19900
 $Comp
-L Antenna AE?
+L Antenna AE1
 U 1 1 5D5A75DA
 P 13900 9350
-F 0 "AE?" H 13825 9425 50  0000 R CNN
+F 0 "AE1" H 13825 9425 50  0000 R CNN
 F 1 "Antenna" H 13825 9350 50  0000 R CNN
 F 2 "" H 13900 9350 50  0001 C CNN
